Commit message: scaled ft_sensor STL, added urdf

File: xarm_description/urdf/ft_sensor/ft_sensor.urdf.xacro (robot description, xacro)
@@ -14,5 +14,5 @@
       <visual>
         <geometry>
-          <mesh filename="file://$(find xarm_description)/meshes/ft_sensor/visual/ft_sensor.STL" scale="0.001 0.001 0.001"/>
+          <mesh filename="file://$(find xarm_description)/meshes/ft_sensor/visual/ft_sensor_scaled.STL"/>
         </geometry>
         <origin xyz="0 0 0" rpy="0 0 0"/>
@@ -21,5 +21,5 @@
       <collision>
         <geometry>
-          <mesh filename="file://$(find xarm_description)/meshes/ft_sensor/collision/ft_sensor.STL" scale="0.001 0.001 0.001"/>
+          <mesh filename="file://$(find xarm_description)/meshes/ft_sensor/collision/ft_sensor_scaled.STL"/>
         </geometry>
         <origin xyz="0 0 0" rpy="0 0 0"/>
