Commit message: fixed no ft sensor urdf, added new urdf file

File: xarm_description/urdf/xarm_device_macro.xacro (robot description, xacro)
@@ -129,10 +129,10 @@
       <xacro:include filename="$(find xarm_description)/urdf/ft_sensor/ft_sensor.urdf.xacro" />
       <xacro:ft_sensor_urdf prefix="${prefix}" />
-    </xacro:if>
-    <joint name="${prefix}joint_ft_sensor" type="fixed">
-      <origin xyz="0 0 0.052" rpy="0 0 -1.5708" />
-      <parent link="${prefix}link${dof}" />
-      <child link="${prefix}link_ft_sensor" />
-    </joint>
+      <joint name="${prefix}joint_ft_sensor" type="fixed">
+        <origin xyz="0 0 0.052" rpy="0 0 -1.5708" />
+        <parent link="${prefix}link${dof}" />
+        <child link="${prefix}link_ft_sensor" />
+      </joint>
+    </xacro:if>
     <xacro:if value="${add_realsense_d435i}">
       <!-- (xarm) Load RealSense D435i URDF -->
