Commit message: updated urdf files to be consistent with feeding repo

File: xarm_description/urdf/xarm6_ft_sensor_gripper.urdf (robot description, URDF)
Before this commit: robot xarm6, 27 links, 26 joints
Links:
- removed link camera_color_frame
- removed link camera_color_optical_frame
- removed link camera_depth_frame
- removed link camera_depth_optical_frame
- removed link camera_left_ir_frame
- removed link camera_left_ir_optical_frame
- removed link camera_link
- removed link camera_right_ir_frame
- removed link camera_right_ir_optical_frame
Joints:
- removed joint camera_color_joint
- removed joint camera_color_optical_joint
- removed joint camera_depth_joint
- removed joint camera_depth_optical_joint
- removed joint camera_left_ir_joint
- removed joint camera_left_ir_optical_joint
- removed joint camera_link_joint
- removed joint camera_right_ir_joint
- removed joint camera_right_ir_optical_joint
- joint joint1: limit lower=-3.1101767270538954 upper=3.1101767270538954 effort=50.0 velocity=3.14 -> lower=-6.283185307179586 upper=6.283185307179586 effort=50.0 velocity=3.14
- joint joint3: limit lower=-3.1101767270538954 upper=0.19198 effort=32.0 velocity=3.14 -> lower=-3.927 upper=0.19198 effort=32.0 velocity=3.14
- joint joint4: limit lower=-3.1101767270538954 upper=3.1101767270538954 effort=32.0 velocity=3.14 -> lower=-6.283185307179586 upper=6.283185307179586 effort=32.0 velocity=3.14
- joint joint5: limit lower=-1.69297 upper=3.1101767270538954 effort=32.0 velocity=3.14 -> lower=-1.69297 upper=3.141592653589793 effort=32.0 velocity=3.14
- joint joint6: limit lower=-3.1101767270538954 upper=3.1101767270538954 effort=20.0 velocity=3.14 -> lower=-6.283185307179586 upper=6.283185307179586 effort=20.0 velocity=3.14

File: xarm_description/urdf/xarm6_with_gripper.urdf (robot description, URDF)
Before this commit: robot xarm6_with_gripper, 17 links, 16 joints
Links:
- link left_finger: geometry collision mesh filename=package://xarm_description/meshes/gripper/xarm/left_finger.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; visual mesh filename=package://xarm_description/meshes/gripper/xarm/left_finger.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
- link left_inner_knuckle: geometry collision mesh filename=package://xarm_description/meshes/gripper/xarm/left_inner_k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; visual mesh filename=package://xarm_description/meshes/gripper/xarm/left_inner_k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
- link left_outer_knuckle: geometry collision mesh filename=package://xarm_description/meshes/gripper/xarm/left_outer_k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; visual mesh filename=package://xarm_description/meshes/gripper/xarm/left_outer_k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
- link link1: mass 2.16 -> 2.3814
- link link2: mass 1.71 -> 2.2675
- link link3: mass 1.384 -> 1.875
- link link4: mass 1.115 -> 1.3192
- link link5: mass 1.275 -> 1.33854
- link link6: mass 0.1096 -> 0.17; geometry collision mesh filename=package://xarm_description/meshes/end_tool/collision/end_to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; visual mesh filename=package://xarm_description/meshes/xarm6/visual/link6.stl
- link link_eef: geometry collision mesh filename=package://xarm_description/meshes/camera/realsense/collisio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; visual mesh filename=package://xarm_description/meshes/camera/realsense/visual/d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
- link right_finger: geometry collision mesh filename=package://xarm_description/meshes/gripper/xarm/right_finger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; visual mesh filename=package://xarm_description/meshes/gripper/xarm/right_finger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
- link right_inner_knuckle: geometry collision mesh filename=package://xarm_description/meshes/gripper/xarm/right_inner_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; visual mesh filename=package://xarm_description/meshes/gripper/xarm/right_inner_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
- link right_outer_knuckle: geometry collision mesh filename=package://xarm_description/meshes/gripper/xarm/right_outer_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; visual mesh filename=package://xarm_description/meshes/gripper/xarm/right_outer_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
- link xarm_gripper_base_link: geometry collision mesh filename=package://xarm_description/meshes/gripper/xarm/base_link.STL; visual mesh filename=package://xarm_description/meshes/gripper/xarm/base_link.STL
Joints:
- joint joint1: limit lower=-6.28318530718 upper=6.28318530718 effort=50.0 velocity=3.14 -> lower=-6.283185307179586 upper=6.283185307179586 effort=50.0 velocity=3.14
- joint joint4: limit lower=-6.28318530718 upper=6.28318530718 effort=32.0 velocity=3.14 -> lower=-6.283185307179586 upper=6.283185307179586 effort=32.0 velocity=3.14
- joint joint5: limit lower=-1.69297 upper=3.14159265359 effort=32.0 velocity=3.14 -> lower=-1.69297 upper=3.141592653589793 effort=32.0 velocity=3.14
- joint joint6: limit lower=-6.28318530718 upper=6.28318530718 effort=20.0 velocity=3.14 -> lower=-6.283185307179586 upper=6.283185307179586 effort=20.0 velocity=3.14
- joint joint_eef: origin xyz=0 0 0 rpy=0 0 0 -> xyz=0 0 0.008 rpy=0 0 0
- joint joint_tcp: origin xyz=0 0 0.122 rpy=0 0 0 -> xyz=0 0 0.152 rpy=0 0 0
