Commit message: added ft sensor and reset config

File: xarm_description/srdf/_xarm6_macro.srdf.xacro (robot description, xacro)
@@ -10,5 +10,5 @@
   <!-- SUBGROUPS: Groups can also be formed by referencing to already defined group names -->
   <xacro:macro name="xarm6_macro_srdf" params="prefix=''
-    add_gripper='false' add_vacuum_gripper='false' add_other_geometry='false' ">
+    add_gripper='false' add_vacuum_gripper='false' add_other_geometry='false' add_ft_sensor='false' ">
     <xacro:if value="${add_gripper}">
       <xacro:property name="_use_gripper" value="true"/>
@@ -85,4 +85,12 @@
       <joint name="${prefix}joint6" value="0" />
     </group_state>
+    <group_state name="reset" group="xarm6">
+      <joint name="${prefix}joint1" value="0" />
+      <joint name="${prefix}joint2" value="0" />
+      <joint name="${prefix}joint3" value="0" />
+      <joint name="${prefix}joint4" value="0" />
+      <joint name="${prefix}joint5" value="-1.3988" />
+      <joint name="${prefix}joint6" value="0" />
+    </group_state>
     <!-- gripper -->
     <xacro:if value="${_use_gripper}">
@@ -112,4 +120,7 @@
       <passive_joint name="${prefix}right_outer_knuckle_joint" />
       <passive_joint name="${prefix}right_finger_joint" />
+      <xacro:if value="${add_ft_sensor}">
+        <passive_joint name="${prefix}joint_ft_sensor" />
+      </xacro:if>
       <!-- DISABLE COLLISIONS, By default it is assumed that any link of the robot could potentially come into collision with any other link in the robot. This tag disables collision checking between a specified pair of links. -->
       <disable_collisions link1="${prefix}left_finger" link2="${prefix}left_inner_knuckle" reason="Default" />
@@ -160,4 +171,13 @@
       <disable_collisions link1="${prefix}link_eef" link2="${prefix}right_inner_knuckle" reason="Never" />
       <disable_collisions link1="${prefix}link_eef" link2="${prefix}right_outer_knuckle" reason="Never" />
+      <xacro:if value="${add_ft_sensor}">
+        <disable_collisions link1="${prefix}link_ft_sensor" link2="${prefix}xarm_gripper_base_link" reason="Adjacent" />
+        <disable_collisions link1="${prefix}link_ft_sensor" link2="${prefix}left_finger" reason="Never" />
+        <disable_collisions link1="${prefix}link_ft_sensor" link2="${prefix}left_inner_knuckle" reason="Never" />
+        <disable_collisions link1="${prefix}link_ft_sensor" link2="${prefix}left_outer_knuckle" reason="Never" />
+        <disable_collisions link1="${prefix}link_ft_sensor" link2="${prefix}right_finger" reason="Never" />
+        <disable_collisions link1="${prefix}link_ft_sensor" link2="${prefix}right_inner_knuckle" reason="Never" />
+        <disable_collisions link1="${prefix}link_ft_sensor" link2="${prefix}right_outer_knuckle" reason="Never" />
+      </xacro:if>
     </xacro:if>
     <!-- vacuum gripper -->
@@ -197,5 +217,12 @@
     <disable_collisions link1="${prefix}link3" link2="${prefix}link_eef" reason="Never" />
     <disable_collisions link1="${prefix}link5" link2="${prefix}link_eef" reason="Never" />
-    <disable_collisions link1="${prefix}link6" link2="${prefix}link_eef" reason="Adjacent" />
+    <xacro:if value="${add_ft_sensor}">
+      <disable_collisions link1="${prefix}link5" link2="${prefix}link_ft_sensor" reason="Never" />
+      <disable_collisions link1="${prefix}link6" link2="${prefix}link_ft_sensor" reason="Adjacent" />
+      <disable_collisions link1="${prefix}link_ft_sensor" link2="${prefix}link_eef" reason="Adjacent" />
+    </xacro:if>
+    <xacro:unless value="${add_ft_sensor}">
+      <disable_collisions link1="${prefix}link6" link2="${prefix}link_eef" reason="Adjacent" />
+    </xacro:unless>
   </xacro:macro>
 </robot>

File: xarm_description/srdf/xarm.srdf.xacro (robot description, xacro)
@@ -6,8 +6,12 @@
   <xacro:arg name="robot_type" default="xarm" />
   <xacro:arg name="add_gripper" default="false"/>
+  <xacro:arg name="add_ft_sensor" default="false" />
   <xacro:arg name="add_vacuum_gripper" default="false" />
   <xacro:arg name="add_other_geometry" default="false" />
   <xacro:include filename="$(find xarm_description)/srdf/xarm_macro.srdf.xacro" />
   <xacro:xarm_macro_srdf prefix="$(arg prefix)" dof="$(arg dof)" robot_type="$(arg robot_type)"
-    add_gripper="$(arg add_gripper)" add_vacuum_gripper="$(arg add_vacuum_gripper)" add_other_geometry="$(arg add_other_geometry)" />
+    add_ft_sensor="$(arg add_ft_sensor)"
+    add_gripper="$(arg add_gripper)"
+    add_vacuum_gripper="$(arg add_vacuum_gripper)"
+    add_other_geometry="$(arg add_other_geometry)" />
 </robot>

File: xarm_description/srdf/xarm_macro.srdf.xacro (robot description, xacro)
@@ -2,5 +2,5 @@
 <robot xmlns:xacro="http://wiki.ros.org/xacro" name="xarm_srdf">
   <xacro:macro name="xarm_macro_srdf" params="prefix:='' dof:=7 robot_type:='xarm'
-    add_gripper:='false' add_vacuum_gripper:='false' add_other_geometry:='false' ">
+    add_gripper:='false' add_vacuum_gripper:='false' add_other_geometry:='false' add_ft_sensor:='false'">
     <xacro:if value="${dof == 5}">
       <xacro:include filename="$(find xarm_description)/srdf/_xarm5_macro.srdf.xacro" />
@@ -17,5 +17,5 @@
         <xacro:include filename="$(find xarm_description)/srdf/_xarm6_macro.srdf.xacro" />
         <xacro:xarm6_macro_srdf prefix="${prefix}"
-          add_gripper="${add_gripper}" add_vacuum_gripper="${add_vacuum_gripper}" add_other_geometry="${add_other_geometry}"  />
+          add_gripper="${add_gripper}" add_ft_sensor="${add_ft_sensor}" add_vacuum_gripper="${add_vacuum_gripper}" add_other_geometry="${add_other_geometry}"  />
       </xacro:unless>
     </xacro:if>

File: xarm_description/urdf/_private_macro.xacro (robot description, xacro)
@@ -2,5 +2,5 @@
 <robot xmlns:xacro="http://ros.org/wiki/xacro" name="private_macro">
   <xacro:property name="is_ros2" value="false" scope="parent"/>
-  <xacro:property name="use_xacro_load_yaml" value="false" scope="parent"/>
+  <xacro:property name="use_xacro_load_yaml" value="true" scope="parent"/>
   <xacro:property name="use_len" value="true" scope="parent"/>
   <xacro:macro name="device_macro_begin" params="">

File: xarm_description/urdf/gripper/xarm_gripper.urdf.xacro (robot description, xacro)
@@ -184,5 +184,5 @@
     <link name="${prefix}link_tcp" />
     <joint name="${prefix}joint_tcp" type="fixed">
-      <origin xyz="0 0 0.172" rpy="0 0 0" />
+      <origin xyz="0 0 0.152" rpy="3.14159 -1.5708 0" />
       <parent link="${prefix}xarm_gripper_base_link" />
       <child link="${prefix}link_tcp" />

File: xarm_description/urdf/xarm_device.urdf.xacro (robot description, xacro)
@@ -16,4 +16,5 @@
   <xacro:arg name="ros2_control_plugin" default="uf_robot_hardware/UFRobotSystemHardware"/>
   <xacro:arg name="ros2_control_params" default="$(find xarm_controller)/config/xarm$(arg dof)_controllers.yaml"/>
+  <xacro:arg name="add_ft_sensor" default="false"/>
   <xacro:arg name="add_realsense_d435i" default="false"/>
   <xacro:arg name="add_d435i_links" default="true"/>
@@ -43,4 +44,5 @@
     ros2_control_plugin="$(arg ros2_control_plugin)" robot_type="$(arg robot_type)"
     load_gazebo_plugin="true" ros2_control_params="$(arg ros2_control_params)"
+    add_ft_sensor="$(arg add_ft_sensor)"
     add_realsense_d435i="$(arg add_realsense_d435i)"
     add_d435i_links="$(arg add_d435i_links)"

File: xarm_description/urdf/xarm_device_macro.xacro (robot description, xacro)
@@ -17,4 +17,5 @@
     ros2_control_params:=''
     load_gazebo_plugin:=false
+    add_ft_sensor:=false
     add_realsense_d435i:=false
     add_d435i_links:=true
@@ -124,4 +125,14 @@
         inertial_params_filename="${inertial_params_filename}" />
     </xacro:unless>
+    <xacro:if value="${add_ft_sensor}">
+      <!-- (xarm) Load 6-axis force-torque sensor URDF -->
+      <xacro:include filename="$(find xarm_description)/urdf/ft_sensor/ft_sensor.urdf.xacro" />
+      <xacro:ft_sensor_urdf prefix="${prefix}" />
+    </xacro:if>
+    <joint name="${prefix}joint_ft_sensor" type="fixed">
+      <origin xyz="0 0 0.052" rpy="0 0 -1.5708" />
+      <parent link="${prefix}link${dof}" />
+      <child link="${prefix}link_ft_sensor" />
+    </joint>
     <xacro:if value="${add_realsense_d435i}">
       <!-- (xarm) Load RealSense D435i URDF -->
@@ -136,9 +147,18 @@
       <link name="${prefix}link_eef"/>
     </xacro:unless>
-    <joint name="${prefix}joint_eef" type="fixed">
-      <origin xyz="0 0 0" rpy="0 0 0" />
-      <parent link="${prefix}link${dof}" />
-      <child link="${prefix}link_eef" />
-    </joint>
+    <xacro:if value="${add_ft_sensor}">
+      <joint name="${prefix}joint_eef" type="fixed">
+        <origin xyz="0 0 0.008" rpy="0 0 1.5708" />
+        <parent link="${prefix}link_ft_sensor" />
+        <child link="${prefix}link_eef" />
+      </joint>
+    </xacro:if>
+    <xacro:unless value="${add_ft_sensor}">
+      <joint name="${prefix}joint_eef" type="fixed">
+        <origin xyz="0 0 0.008" rpy="0 0 0" />
+        <parent link="${prefix}link${dof}" />
+        <child link="${prefix}link_eef" />
+      </joint>
+    </xacro:unless>
     <xacro:if value="${add_gripper}">
       <xacro:if value="${robot_type == 'lite'}">

File: xarm_gripper/urdf/xarm_gripper.urdf.xacro (robot description, xacro)
@@ -402,5 +402,5 @@
     <origin
       xyz="0 0 0.172"
-      rpy="0 0 0" />
+      rpy="3.14159 -1.5708 0" />
     <parent
       link="${prefix}xarm_gripper_base_link" />

Commit message: add new named state

File: xarm_description/srdf/_xarm6_macro.srdf.xacro (robot description, xacro)
@@ -92,4 +92,12 @@
       <joint name="${prefix}joint5" value="-1.3988" />
       <joint name="${prefix}joint6" value="0" />
+    </group_state>
+    <group_state group="xarm6" name="goal_gen">
+      <joint name="joint1" value="0"/>
+      <joint name="joint2" value="-0.5988722443580627"/>
+      <joint name="joint3" value="0.023431047797203064"/>
+      <joint name="joint4" value="0"/>
+      <joint name="joint5" value="-0.5772890448570251"/>
+      <joint name="joint6" value="0"/>
     </group_state>
     <!-- gripper -->
